File: ESP32-H2/matter-thread/matter-button-cr2032/hardware/matter-button-cr2032.kicad_sch (KiCad schematic)
At the start: 37 parts, among them Q1 DMG2305UX, SW1 PTS810, U1 ESP32-H2-WROOM-02C-H4S, U2 TPS63900DSKR

Commit message: matter-button-cr2032: JLCPCB Basic parts and LCSC part numbers
Every assembled part now carries an LCSC part number (schematic field,
footprint field, BOM). Common parts moved to the JLCPCB Basic library:
- Q1 AO3401A (C15127) instead of DMG2305UX, same SOT-23 pinout
- D1 KT-0603R (C2286), passives UNI-ROYAL / Samsung Basic parts
- R3 (CFG3) 0 ohm as the TI 3.3 V reference design: VO(1) = 1.8 V,
  unused because SEL is tied to VIN; R2 and R3 share one part
- R6 button pull-up 1 Mohm (same part as R9): 3.3 uA while pressed
Extended parts left: U2, L1 (DFE252012P-2R2M), C1/C2, R1 36.5k, SW1
(PTS810 SJM, 160 gf). U1 and BT1 are not stocked by LCSC: left out of
the JLCPCB BOM and CPL, hand soldered.

gen_pcb.py sync updates values and part fields on the routed board
without placement or routing. Copper and Gerbers are unchanged;
ERC 0, DRC 0 with schematic parity.

Co-Authored-By: Claude Opus 5.5 <noreply@anthropic.com>
Claude-Session: https://claude.ai/code/session_01R15P3zWK2KCijMWrCL7LHn
Parts:
- C1, C2: LCSC (none) -> C469553
- C3, C5: LCSC (none) -> C19702; MPN GRM188R61A106ME69D -> CL10A106KP8NNNC
- C4: LCSC (none) -> C59461; MPN GRM187R60J226ME15D -> CL10A226MQ8NRNC
- C6, C9: LCSC (none) -> C1525; MPN GRM155R71C104KA88D -> CL05B104KO5NNNC
- C7: LCSC (none) -> C52923; MPN GRM155R61A105KE15D -> CL05A105KA5NQNC
- C8: LCSC (none) -> C1523; MPN GRM155R71H102KA01D -> CL05B102KB5NNNC
- D1: LCSC (none) -> C2286; MPN KP-1608SURCK -> KT-0603R
- L1: LCSC (none) -> C391305; MPN DFE252012F-2R2M=P2 -> DFE252012P-2R2M=P2
- Q1: value DMG2305UX -> AO3401A; LCSC (none) -> C15127; MPN DMG2305UX-7 -> AO3401A
- R1: LCSC (none) -> C49010116; MPN RC0402FR-0736K5L -> FRC0402F3652TS
- R2: LCSC (none) -> C17168; MPN RC0402JR-070RL -> 0402WGF0000TCE
- R3: value 16.2k -> 0R; LCSC (none) -> C17168; MPN RC0402FR-0716K2L -> 0402WGF0000TCE
- R4, R5: LCSC (none) -> C25744; MPN RC0402FR-0710KL -> 0402WGF1002TCE
- R6: value 470k -> 1M; LCSC (none) -> C26083; MPN RC0402FR-07470KL -> 0402WGF1004TCE
- R7, R8: LCSC (none) -> C11702; MPN RC0402FR-071KL -> 0402WGF1001TCE
- R9: LCSC (none) -> C26083; MPN RC0402FR-071ML -> 0402WGF1004TCE
- SW1: LCSC (none) -> C116501
- U2: LCSC (none) -> C1518762
Other:
- note added: "CFG1 36.5k + CFG2 0R: VO(2) = 3.3 V, no input current limit; CFG3 0R: VO(1) = 1.8 V, unused: EN, SEL to VIN"
- note removed: "CFG1 36.5k + CFG2 0R: VO(2) = 3.3 V, no input current limit; CFG3 16.2k: VO(1) = 3.3 V; EN, SEL to VIN"
